File: layout.sch (KiCad schematic (older format))
At the start: 1 part

Commit message: _schema
Parts:
- added C?: CSMALL, symbol CSMALL
- added C?: C, symbol C
- added C? (x2): 15p, symbol CSMALL
- added D?: LED, symbol LED
- added J?: USB_2, symbol USB_2
- added Q? (x2): MOS_N, symbol MOS_N
- added Q?: MOSFET_P, symbol MOSFET_P
- added R?: R, symbol R
- added SW?: SW_PUSH, symbol SW_PUSH
- added U?: PHTRANS, symbol PHTRANS
- added U?: PHDARL, symbol PHDARL
- added X?: CRYSTAL, symbol CRYSTAL
- added X?: CRYSTAL 12MHz, symbol CRYSTAL
Connections:
- wire segments 0 -> 8
Changed lines of the file:
@@
-EESchema Schematic File Version 2  date Po 14. březen 2016, 13:02:18 CET
+EESchema Schematic File Version 2  date Po 14. březen 2016, 17:50:40 CET
 LIBS:power
 LIBS:device
@@
 LIBS:contrib
 LIBS:valves
-EELAYER 43  0
+LIBS:layout-cache
+EELAYER 25  0
 EELAYER END
 $Descr A4 11700 8267
@@
 Comment4 ""
 $EndDescr
+Connection ~ 3800 3700
+Wire Wire Line
+	3700 3700 4400 3700
+Wire Wire Line
+	3700 3700 3700 2800
+Wire Wire Line
+	3700 2800 4400 2800
+Connection ~ 3800 3300
+Wire Wire Line
+	3800 3500 3800 3100
+Wire Wire Line
+	3800 3100 4400 3100
+Wire Wire Line
+	4400 3500 4400 3300
+Wire Wire Line
+	4400 3700 4400 5000
+Wire Wire Line
+	4400 5000 5300 5000
+$Comp
+L CSMALL C?
+U 1 1 56E6EA03
+P 4400 3600
+F 0 "C?" H 4425 3650 30  0000 L CNN
+F 1 "15p" H 4425 3550 30  0000 L CNN
+	1    4400 3600
+	1    0    0    -1
+$EndComp
+$Comp
+L CSMALL C?
+U 1 1 56E6E9FE
+P 3800 3600
+F 0 "C?" H 3825 3650 30  0000 L CNN
+F 1 "15p" H 3825 3550 30  0000 L CNN
+	1    3800 3600
+	1    0    0    -1
+$EndComp
+$Comp
+L CRYSTAL X?
+U 1 1 56E6E934
+P 4100 3300
+F 0 "X?" H 4100 3450 60  0000 C CNN
+F 1 "CRYSTAL 12MHz" H 4100 3150 40  0000 C CNN
+	1    4100 3300
+	1    0    0    -1
+$EndComp
+$Comp
+L C C?
+U 1 1 56E6E8CC
+P 10800 3650
+F 0 "C?" H 10850 3750 50  0000 L CNN
+F 1 "C" H 10850 3550 50  0000 L CNN
+	1    10800 3650
+	1    0    0    -1
+$EndComp
+$Comp
+L CRYSTAL X?
+U 1 1 56E6E8B3
+P 10750 2950
+F 0 "X?" H 10750 3100 60  0000 C CNN
+F 1 "CRYSTAL" H 10750 2800 60  0000 C CNN
+	1    10750 2950
+	1    0    0    -1
+$EndComp
+$Comp
+L CSMALL C?
+U 1 1 56E6E8A6
+P 10800 2350
+F 0 "C?" H 10825 2400 30  0000 L CNN
+F 1 "CSMALL" H 10825 2300 30  0000 L CNN
+	1    10800 2350
+	1    0    0    -1
+$EndComp
+$Comp
+L MOSFET_P Q?
+U 1 1 56E6E848
+P 10850 1600
+F 0 "Q?" H 10850 1790 60  0000 R CNN
+F 1 "MOSFET_P" H 10850 1420 60  0000 R CNN
+	1    10850 1600
+	1    0    0    -1
+$EndComp
+$Comp
+L MOS_N Q?
+U 1 1 56E6E837
+P 10850 900
+F 0 "Q?" H 10860 1070 60  0000 R CNN
+F 1 "MOS_N" H 10860 750 60  0000 R CNN
+	1    10850 900
+	1    0    0    -1
+$EndComp
+$Comp
+L PHDARL U?
+U 1 1 56E6E80F
+P 10300 6350
+F 0 "U?" H 10310 6670 70  0000 C CNN
+F 1 "PHDARL" H 10310 6030 70  0000 C CNN
+	1    10300 6350
+	1    0    0    -1
+$EndComp
+$Comp
+L PHTRANS U?
+U 1 1 56E6E7FF
+P 8650 6350
+F 0 "U?" H 8600 6700 70  0000 C CNN
+F 1 "PHTRANS" H 8600 6000 70  0000 C CNN
+	1    8650 6350
+	1    0    0    -1
+$EndComp
+$Comp
+L R R?
+U 1 1 56E6E7CF
+P 9050 3350
+F 0 "R?" V 9130 3350 50  0000 C CNN
+F 1 "R" V 9050 3350 50  0000 C CNN
+	1    9050 3350
+	1    0    0    -1
+$EndComp
+$Comp
+L SW_PUSH SW?
+U 1 1 56E6E7A3
+P 8850 2750
+F 0 "SW?" H 9000 2860 50  0000 C CNN
+F 1 "SW_PUSH" H 8850 2670 50  0000 C CNN
+	1    8850 2750
+	1    0    0    -1
+$EndComp
+$Comp
+L MOS_N Q?
+U 1 1 56E6E758
+P 8900 2150
+F 0 "Q?" H 8910 2320 60  0000 R CNN
+F 1 "MOS_N" H 8910 2000 60  0000 R CNN
+	1    8900 2150
+	1    0    0    -1
+$EndComp
+$Comp
+L LED D?
+U 1 1 56E6E6FA
+P 8000 2200
+F 0 "D?" H 8000 2300 50  0000 C CNN
+F 1 "LED" H 8000 2100 50  0000 C CNN
+	1    8000 2200
+	1    0    0    -1
+$EndComp
+$Comp
+L USB_2 J?
+U 1 1 56E6E639
+P 3000 1900
+F 0 "J?" H 2925 2150 60  0000 C CNN
+F 1 "USB_2" H 3050 1600 60  0001 C CNN
+F 4 "VCC" H 3325 2050 50  0001 C CNN "VCC"
+F 5 "D+" H 3300 1950 50  0001 C CNN "Data+"
+F 6 "D-" H 3300 1850 50  0001 C CNN "Data-"
+F 7 "GND" H 3325 1750 50  0001 C CNN "Ground"
+	1    3000 1900
+	1    0    0    -1
+$EndComp
 $Comp
 L ATMEGA8-P IC?

Commit message: _schema
Parts:
- removed C?: CSMALL, symbol CSMALL
- removed C?: C, symbol C
- removed D?: LED, symbol LED
- removed J?: USB_2, symbol USB_2
- removed Q? (x2): MOS_N, symbol MOS_N
- removed Q?: MOSFET_P, symbol MOSFET_P
- removed R?: R, symbol R
- removed SW?: SW_PUSH, symbol SW_PUSH
- removed U?: PHTRANS, symbol PHTRANS
- removed U?: PHDARL, symbol PHDARL
- removed X?: CRYSTAL, symbol CRYSTAL
- added C? (x2): 15p, symbol CSMALL
- added C?: 1uF, symbol CP1
- added D?: LED, symbol LED
- added IC?: ATMEGA8-P, DIL28, symbol ATMEGA8-P
- added J?: externí zdroj 5V, symbol USB_2
- added J?: USB_2, symbol USB_2
- added JP?: JUMPER-slow_sck, symbol JUMPER
- added R? (x2): 10k, symbol R
- added R? (x2): 470, symbol R
- added R?: 1k5, symbol R
- added X?: CRYSTAL 12MHz, symbol CRYSTAL
- C? (x2): value 15p -> 33p
Connections:
- net labels added: +5V, Basic usb_asp programmer with apl. circuit - atmega8, GND, Usb external power supply - 5V / 100mA, Usb for PC programming
- wire segments 8 -> 53
Other:
- moved on the sheet: IC?, X?

Commit message: sch_net_pcb_proj
Parts:
- gave numbers to parts that had none: 18
Connections:
- net labels removed: +5V
- wire segments 53 -> 56
Other:
- moved on the sheet: C1, D1, R1

Commit message: sch_net_pcb_proj
Parts:
- added P1: CONN_6, symbol CONN_6
Connections:
- wire segments 56 -> 62
Changed lines of the file:
@@
-EESchema Schematic File Version 2  date Út 15. březen 2016, 14:11:44 CET
+EESchema Schematic File Version 2  date Čt 17. březen 2016, 15:31:34 CET
 LIBS:power
 LIBS:device
@@
 Sheet 1 1
 Title ""
-Date "15 mar 2016"
+Date "17 mar 2016"
 Rev ""
 Comp ""
@@
 Comment4 ""
 $EndDescr
+$Comp
+L CONN_6 P1
+U 1 1 56EABEA5
+P 4250 5650
+F 0 "P1" V 4200 5650 60  0000 C CNN
+F 1 "CONN_6" V 4300 5650 60  0000 C CNN
+	1    4250 5650
+	1    0    0    -1
+$EndComp
+Wire Wire Line
+	3600 5900 3900 5900
+Wire Wire Line
+	3600 5700 3900 5700
+Wire Wire Line
+	3600 5500 3900 5500
 Wire Wire Line
 	1450 4950 1400 4950
@@
 	950  5000 900  5000
 Connection ~ 900  5000
+Wire Wire Line
+	3600 5400 3900 5400
+Wire Wire Line
+	3600 5600 3900 5600
+Wire Wire Line
+	3600 5800 3900 5800
 Text Label 8550 7350 0    60   ~ 0
 Basic usb_asp programmer with apl. circuit - atmega8
 $Comp
-L GND #PWR01
+L GND #PWR5
 U 1 1 56E6FC1F
 P 5900 4900
-F 0 "#PWR01" H 5900 4900 30  0001 C CNN
+F 0 "#PWR5" H 5900 4900 30  0001 C CNN
 F 1 "GND" H 5900 4830 30  0001 C CNN
 	1    5900 4900
@@
 $EndComp
 $Comp
-L GND #PWR02
+L GND #PWR3
 U 1 1 56E6F74F
 P 5700 2500
-F 0 "#PWR02" H 5700 2500 30  0001 C CNN
+F 0 "#PWR3" H 5700 2500 30  0001 C CNN
 F 1 "GND" H 5700 2430 30  0001 C CNN
 	1    5700 2500
@@
 $EndComp
 $Comp
-L GND #PWR03
+L GND #PWR4
 U 1 1 56E6F4BB
 P 5900 1600
-F 0 "#PWR03" H 5900 1600 30  0001 C CNN
+F 0 "#PWR4" H 5900 1600 30  0001 C CNN
 F 1 "GND" H 5900 1530 30  0001 C CNN
 	1    5900 1600
@@
 $EndComp
 $Comp
-L GND #PWR04
+L GND #PWR1
 U 1 1 56E6EE76
 P 2600 4150
-F 0 "#PWR04" H 2600 4150 30  0001 C CNN
+F 0 "#PWR1" H 2600 4150 30  0001 C CNN
 F 1 "GND" H 2600 4080 30  0001 C CNN
 	1    2600 4150
@@
 $EndComp
 $Comp
-L GND #PWR05
+L GND #PWR2
 U 1 1 56E6ED32
 P 2600 7400
-F 0 "#PWR05" H 2600 7400 30  0001 C CNN
+F 0 "#PWR2" H 2600 7400 30  0001 C CNN
 F 1 "GND" H 2600 7330 30  0001 C CNN
 	1    2600 7400

Commit message: sch_net_pcb_proj
Parts:
- added P? (x2): CONN_5, symbol CONN_5
- added P?: CONN_4, symbol CONN_4
Connections:
- wire segments 62 -> 74
Other:
- moved on the sheet: D1
Changed lines of the file:
@@
-EESchema Schematic File Version 2  date Čt 17. březen 2016, 15:31:34 CET
+EESchema Schematic File Version 2  date So 19. březen 2016, 18:29:40 CET
 LIBS:power
 LIBS:device
@@
 Sheet 1 1
 Title ""
-Date "17 mar 2016"
+Date "19 mar 2016"
 Rev ""
 Comp ""
@@
 Comment4 ""
 $EndDescr
+Wire Wire Line
+	3850 4800 3600 4800
+Connection ~ 3700 5000
+Wire Wire Line
+	3850 5000 3600 5000
+Connection ~ 3800 5200
+Wire Wire Line
+	3850 5200 3600 5200
+Wire Wire Line
+	3600 6800 3900 6800
+Wire Wire Line
+	3600 6600 3900 6600
+Wire Wire Line
+	3600 6400 3850 6400
+Wire Wire Line
+	3600 6200 3850 6200
+Connection ~ 1450 4400
+Wire Wire Line
+	1450 4500 1450 4400
+Connection ~ 900  4400
+Connection ~ 2600 4400
+Wire Wire Line
+	3600 5900 3900 5900
+Wire Wire Line
+	3600 5700 3900 5700
+Wire Wire Line
+	3600 5500 3900 5500
+Wire Wire Line
+	900  4450 900  1150
+Wire Wire Line
+	5900 4700 5900 4900
+Wire Wire Line
+	3600 3050 4300 3050
+Wire Wire Line
+	4900 1650 5000 1650
+Wire Wire Line
+	5000 1650 5000 1350
+Wire Wire Line
+	3800 5200 3800 1950
+Wire Wire Line
+	3800 1950 3600 1950
+Wire Wire Line
+	3700 5000 3700 1750
+Wire Wire Line
+	3700 1750 3600 1750
+Wire Wire Line
+	4300 3050 4300 1550
+Wire Wire Line
+	4300 1550 3600 1550
+Wire Wire Line
+	5700 2350 5700 2500
+Wire Wire Line
+	5000 1350 5900 1350
+Wire Wire Line
+	4900 1450 4900 1250
+Connection ~ 4400 1150
+Wire Wire Line
+	4400 1150 4400 1250
+Connection ~ 2600 1150
+Wire Wire Line
+	900  1150 5900 1150
+Wire Wire Line
+	2600 4150 2600 4050
+Connection ~ 1100 2750
+Wire Wire Line
+	1000 2750 1700 2750
+Wire Wire Line
+	1000 2750 1000 1850
+Wire Wire Line
+	1000 1850 1700 1850
+Connection ~ 1100 2350
+Wire Wire Line
+	1100 2550 1100 2150
+Wire Wire Line
+	1700 2350 1700 2550
+Wire Wire Line
+	1700 7300 1700 6000
+Wire Wire Line
+	1700 5800 1700 5600
+Wire Wire Line
+	1700 5400 1100 5400
+Wire Wire Line
+	1100 5400 1100 5800
+Connection ~ 1100 5600
+Wire Wire Line
+	1700 5100 1000 5100
+Wire Wire Line
+	1000 5100 1000 6000
+Wire Wire Line
+	1000 6000 1700 6000
+Connection ~ 1100 6000
+Wire Wire Line
+	1100 2150 1700 2150
+Wire Wire Line
+	1700 2750 1700 4050
+Wire Wire Line
+	1700 4050 2600 4050
+Wire Wire Line
+	2600 7400 2600 7300
+Wire Wire Line
+	5900 1450 5900 1600
+Wire Wire Line
+	4900 1250 5900 1250
+Wire Wire Line
+	4400 1450 3600 1450
+Wire Wire Line
+	1200 1150 1200 1450
+Connection ~ 1200 1150
+Wire Wire Line
+	5100 2350 3600 2350
+Wire Wire Line
+	1700 4700 1700 4300
+Wire Wire Line
+	3600 1850 3750 1850
+Wire Wire Line
+	3750 1850 3750 5100
+Wire Wire Line
+	3600 1650 4000 1650
+Wire Wire Line
+	4000 1650 4000 4300
+Wire Wire Line
+	4000 4300 1700 4300
+Wire Wire Line
+	4400 1650 4300 1650
+Connection ~ 4300 1650
+Wire Wire Line
+	900  4800 900  7300
+Wire Wire Line
+	900  7300 2600 7300
+Connection ~ 1700 7300
+Wire Wire Line
+	900  4400 5900 4400
+Wire Wire Line
+	950  5000 900  5000
+Connection ~ 900  5000
+Wire Wire Line
+	3600 5400 3900 5400
+Wire Wire Line
+	3600 5600 3900 5600
+Wire Wire Line
+	3600 5800 3900 5800
+Wire Wire Line
+	1450 5000 1450 4900
+Wire Wire Line
+	3600 6100 3850 6100
+Wire Wire Line
+	3600 6300 3850 6300
+Wire Wire Line
+	3600 6500 3850 6500
+Wire Wire Line
+	3600 6700 3900 6700
+Wire Wire Line
+	3900 6900 3900 7050
+Wire Wire Line
+	3900 7050 4450 7050
+Wire Wire Line
+	4450 7050 4450 4700
+Wire Wire Line
+	4450 4700 3600 4700
+Wire Wire Line
+	3850 5100 3600 5100
+Connection ~ 3750 5100
+Wire Wire Line
+	3850 4900 3600 4900
+$Comp
+L CONN_5 P?
+U 1 1 56ED8B75
+P 4250 5000
+F 0 "P?" V 4200 5000 50  0000 C CNN
+F 1 "CONN_5" V 4300 5000 50  0000 C CNN
+	1    4250 5000
+	1    0    0    -1
+$EndComp
+$Comp
+L CONN_4 P?
+U 1 1 56ED8B6B
+P 4250 6750
+F 0 "P?" V 4200 6750 50  0000 C CNN
+F 1 "CONN_4" V 4300 6750 50  0000 C CNN
+	1    4250 6750
+	1    0    0    -1
+$EndComp
+$Comp
+L CONN_5 P?
+U 1 1 56ED8A65
+P 4250 6300
+F 0 "P?" V 4200 6300 50  0000 C CNN
+F 1 "CONN_5" V 4300 6300 50  0000 C CNN
+	1    4250 6300
+	1    0    0    -1
+$EndComp
 $Comp
 L CONN_6 P1
@@
 	1    0    0    -1
 $EndComp
-Wire Wire Line
-	3600 5900 3900 5900
-Wire Wire Line
-	3600 5700 3900 5700
-Wire Wire Line
-	3600 5500 3900 5500
-Wire Wire Line
-	1450 4950 1400 4950
-Wire Wire Line
-	1450 4950 1450 5000
-Connection ~ 900  4400
-Wire Wire Line
-	900  4450 900  1150
-Wire Wire Line
-	5900 4700 5900 4900
-Wire Wire Line
-	1400 4950 1400 4800
-Wire Wire Line
-	3600 3050 4300 3050
-Wire Wire Line
-	4900 1650 5000 1650
-Wire Wire Line
-	5000 1650 5000 1350
-Wire Wire Line
-	3600 5200 3900 5200
-Wire Wire Line
-	3900 5200 3900 1950
-Wire Wire Line
-	3900 1950 3600 1950
-Wire Wire Line
-	3600 5000 3700 5000
-Wire Wire Line
-	3700 5000 3700 1750
-Wire Wire Line
-	3700 1750 3600 1750
-Wire Wire Line
-	4300 3050 4300 1550
-Wire Wire Line
-	4300 1550 3600 1550
-Wire Wire Line
-	5700 2350 5700 2500
-Wire Wire Line
-	5000 1350 5900 1350
-Wire Wire Line
-	4900 1450 4900 1250
-Connection ~ 4400 1150
-Wire Wire Line
-	4400 1250 4400 1150
-Connection ~ 2600 1150
-Wire Wire Line
-	900  1150 5900 1150
-Wire Wire Line
-	2600 4150 2600 4050
-Connection ~ 1100 2750
-Wire Wire Line
-	1000 2750 1700 2750
-Wire Wire Line
-	1000 2750 1000 1850
-Wire Wire Line
-	1000 1850 1700 1850
-Connection ~ 1100 2350
-Wire Wire Line
-	1100 2550 1100 2150
-Wire Wire Line
-	1700 2350 1700 2550
-Wire Wire Line
-	1700 7300 1700 6000
-Wire Wire Line
-	1700 5800 1700 5600
-Wire Wire Line
-	1700 5400 1100 5400
-Wire Wire Line
-	1100 5400 1100 5800
-Connection ~ 1100 5600
-Wire Wire Line
-	1700 5100 1000 5100
-Wire Wire Line
-	1000 5100 1000 6000
-Wire Wire Line
-	1000 6000 1700 6000
-Connection ~ 1100 6000
-Wire Wire Line
-	1100 2150 1700 2150
-Wire Wire Line
-	1700 2750 1700 4050
-Wire Wire Line
-	1700 4050 2600 4050
-Wire Wire Line
-	2600 7400 2600 7300
-Wire Wire Line
-	5900 1450 5900 1600
-Wire Wire Line
-	4900 1250 5900 1250
-Wire Wire Line
-	4400 1450 3600 1450
-Wire Wire Line
-	1200 1450 1200 1150
-Connection ~ 1200 1150
-Wire Wire Line
-	5100 2350 3600 2350
-Wire Wire Line
-	1700 4700 1700 4300
-Wire Wire Line
-	3600 1850 3800 1850
-Wire Wire Line
-	3800 1850 3800 5100
-Wire Wire Line
-	3800 5100 3600 5100
-Wire Wire Line
-	3600 1650 4000 1650
-Wire Wire Line
-	4000 1650 4000 4300
-Wire Wire Line
-	4000 4300 1700 4300
-Wire Wire Line
-	4400 1650 4300 1650
-Connection ~ 4300 1650
-Wire Wire Line
-	900  4800 900  7300
-Wire Wire Line
-	900  7300 2600 7300
-Connection ~ 1700 7300
-Wire Wire Line
-	900  4400 5900 4400
-Connection ~ 2600 4400
-Wire Wire Line
-	1400 4500 1400 4400
-Connection ~ 1400 4400
-Wire Wire Line
-	950  5000 900  5000
-Connection ~ 900  5000
-Wire Wire Line
-	3600 5400 3900 5400
-Wire Wire Line
-	3600 5600 3900 5600
-Wire Wire Line
-	3600 5800 3900 5800
 Text Label 8550 7350 0    60   ~ 0
 Basic usb_asp programmer with apl. circuit - atmega8
@@
 L LED D1
 U 1 1 56E6FAF2
-P 1400 4700
-F 0 "D1" H 1400 4800 50  0000 C CNN
-F 1 "LED" H 1400 4600 50  0000 C CNN
-	1    1400 4700
+P 1450 4700
+F 0 "D1" H 1450 4800 50  0000 C CNN
+F 1 "LED" H 1450 4600 50  0000 C CNN
+	1    1450 4700
 	0    -1   1    0
 $EndComp

Commit message: updated at >>
Parts:
- gave numbers to parts that had none: 3
Changed lines of the file:
@@
-EESchema Schematic File Version 2  date So 19. březen 2016, 18:29:40 CET
+EESchema Schematic File Version 2  date Ne 20. březen 2016, 19:17:08 CET
 LIBS:power
 LIBS:device
@@
 	3850 4900 3600 4900
 $Comp
-L CONN_5 P?
+L CONN_5 P2
 U 1 1 56ED8B75
 P 4250 5000
-F 0 "P?" V 4200 5000 50  0000 C CNN
+F 0 "P2" V 4200 5000 50  0000 C CNN
 F 1 "CONN_5" V 4300 5000 50  0000 C CNN
 	1    4250 5000
@@
 $EndComp
 $Comp
-L CONN_4 P?
+L CONN_4 P4
 U 1 1 56ED8B6B
 P 4250 6750
-F 0 "P?" V 4200 6750 50  0000 C CNN
+F 0 "P4" V 4200 6750 50  0000 C CNN
 F 1 "CONN_4" V 4300 6750 50  0000 C CNN
 	1    4250 6750
@@
 $EndComp
 $Comp
-L CONN_5 P?
+L CONN_5 P3
 U 1 1 56ED8A65
 P 4250 6300
-F 0 "P?" V 4200 6300 50  0000 C CNN
+F 0 "P3" V 4200 6300 50  0000 C CNN
 F 1 "CONN_5" V 4300 6300 50  0000 C CNN
 	1    4250 6300

Commit message: updated at >>
Parts:
- added K? (x2): CONN_3, symbol CONN_3
Connections:
- wire segments 74 -> 77
Changed lines of the file:
@@
-EESchema Schematic File Version 2  date Ne 20. březen 2016, 19:17:08 CET
+EESchema Schematic File Version 2  date Po 21. březen 2016, 16:43:15 CET
 LIBS:power
 LIBS:device
@@
 Sheet 1 1
 Title ""
-Date "19 mar 2016"
+Date "21 mar 2016"
 Rev ""
 Comp ""
@@
 $EndDescr
 Wire Wire Line
+	3700 5000 3700 3950
+Wire Wire Line
+	3700 3950 3900 3950
+Wire Wire Line
+	3800 5200 3800 4150
+Wire Wire Line
+	3800 4150 3900 4150
+Wire Wire Line
+	3600 1850 3800 1850
+Wire Wire Line
+	3850 4900 3600 4900
+Connection ~ 3750 5100
+Wire Wire Line
+	3850 5100 3600 5100
+Wire Wire Line
+	3600 4700 4450 4700
+Wire Wire Line
+	4450 4700 4450 7050
+Wire Wire Line
+	4450 7050 3900 7050
+Wire Wire Line
+	3900 7050 3900 6900
+Wire Wire Line
+	3600 6700 3900 6700
+Wire Wire Line
+	3600 6500 3850 6500
+Wire Wire Line
+	3600 6300 3850 6300
+Wire Wire Line
+	3600 6100 3850 6100
+Wire Wire Line
+	1450 5000 1450 4900
+Wire Wire Line
+	3600 5800 3900 5800
+Wire Wire Line
+	3600 5600 3900 5600
+Wire Wire Line
+	3600 5400 3900 5400
+Connection ~ 900  5000
+Wire Wire Line
+	950  5000 900  5000
+Wire Wire Line
+	900  4400 5900 4400
+Connection ~ 1700 7300
+Wire Wire Line
+	900  7300 2600 7300
+Wire Wire Line
+	900  7300 900  4800
+Connection ~ 4300 1650
+Wire Wire Line
+	4400 1650 4300 1650
+Wire Wire Line
+	4000 4300 1700 4300
+Wire Wire Line
+	4000 4300 4000 1650
+Wire Wire Line
+	4000 1650 3600 1650
+Wire Wire Line
+	1700 4300 1700 4700
+Wire Wire Line
+	5100 2350 3600 2350
+Connection ~ 1200 1150
+Wire Wire Line
+	1200 1150 1200 1450
+Wire Wire Line
+	4400 1450 3600 1450
+Wire Wire Line
+	5900 1250 4900 1250
+Wire Wire Line
+	5900 1450 5900 1600
+Wire Wire Line
+	2600 7300 2600 7400
+Wire Wire Line
+	1700 4050 2600 4050
+Wire Wire Line
+	1700 4050 1700 2750
+Wire Wire Line
+	1700 2150 1100 2150
+Connection ~ 1100 6000
+Wire Wire Line
+	1000 6000 1700 6000
+Wire Wire Line
+	1000 6000 1000 5100
+Wire Wire Line
+	1000 5100 1700 5100
+Connection ~ 1100 5600
+Wire Wire Line
+	1100 5800 1100 5400
+Wire Wire Line
+	1100 5400 1700 5400
+Wire Wire Line
+	1700 5800 1700 5600
+Wire Wire Line
+	1700 6000 1700 7300
+Wire Wire Line
+	1700 2350 1700 2550
+Wire Wire Line
+	1100 2150 1100 2550
+Connection ~ 1100 2350
+Wire Wire Line
+	1700 1850 1000 1850
+Wire Wire Line
+	1000 1850 1000 2750
+Wire Wire Line
+	1000 2750 1700 2750
+Connection ~ 1100 2750
+Wire Wire Line
+	2600 4050 2600 4150
+Wire Wire Line
+	5900 1150 900  1150
+Connection ~ 2600 1150
+Wire Wire Line
+	4400 1150 4400 1250
+Connection ~ 4400 1150
+Wire Wire Line
+	4900 1250 4900 1450
+Wire Wire Line
+	5900 1350 5000 1350
+Wire Wire Line
+	5700 2350 5700 2500
+Wire Wire Line
+	3600 1550 4300 1550
+Wire Wire Line
+	4300 1550 4300 3050
+Wire Wire Line
+	5000 1350 5000 1650
+Wire Wire Line
+	5000 1650 4900 1650
+Wire Wire Line
+	4300 3050 3600 3050
+Wire Wire Line
+	5900 4700 5900 4900
+Wire Wire Line
+	900  1150 900  4450
+Wire Wire Line
+	3600 5500 3900 5500
+Wire Wire Line
+	3600 5700 3900 5700
+Wire Wire Line
+	3600 5900 3900 5900
+Connection ~ 2600 4400
+Connection ~ 900  4400
+Wire Wire Line
+	1450 4500 1450 4400
+Connection ~ 1450 4400
+Wire Wire Line
+	3600 6200 3850 6200
+Wire Wire Line
+	3600 6400 3850 6400
+Wire Wire Line
+	3600 6600 3900 6600
+Wire Wire Line
+	3600 6800 3900 6800
+Wire Wire Line
+	3850 5200 3600 5200
+Connection ~ 3800 5200
+Wire Wire Line
+	3850 5000 3600 5000
+Connection ~ 3700 5000
+Wire Wire Line
 	3850 4800 3600 4800
-Connection ~ 3700 5000
-Wire Wire Line
-	3850 5000 3600 5000
-Connection ~ 3800 5200
-Wire Wire Line
-	3850 5200 3600 5200
-Wire Wire Line
-	3600 6800 3900 6800
-Wire Wire Line
-	3600 6600 3900 6600
-Wire Wire Line
-	3600 6400 3850 6400
-Wire Wire Line
-	3600 6200 3850 6200
-Connection ~ 1450 4400
-Wire Wire Line
-	1450 4500 1450 4400
-Connection ~ 900  4400
-Connection ~ 2600 4400
-Wire Wire Line
-	3600 5900 3900 5900
-Wire Wire Line
-	3600 5700 3900 5700
-Wire Wire Line
-	3600 5500 3900 5500
-Wire Wire Line
-	900  4450 900  1150
-Wire Wire Line
-	5900 4700 5900 4900
-Wire Wire Line
-	3600 3050 4300 3050
-Wire Wire Line
-	4900 1650 5000 1650
-Wire Wire Line
-	5000 1650 5000 1350
-Wire Wire Line
-	3800 5200 3800 1950
-Wire Wire Line
-	3800 1950 3600 1950
-Wire Wire Line
-	3700 5000 3700 1750
-Wire Wire Line
-	3700 1750 3600 1750
-Wire Wire Line
-	4300 3050 4300 1550
-Wire Wire Line
-	4300 1550 3600 1550
-Wire Wire Line
-	5700 2350 5700 2500
-Wire Wire Line
-	5000 1350 5900 1350
-Wire Wire Line
-	4900 1450 4900 1250
-Connection ~ 4400 1150
-Wire Wire Line
-	4400 1150 4400 1250
-Connection ~ 2600 1150
-Wire Wire Line
-	900  1150 5900 1150
-Wire Wire Line
-	2600 4150 2600 4050
-Connection ~ 1100 2750
-Wire Wire Line
-	1000 2750 1700 2750
-Wire Wire Line
-	1000 2750 1000 1850
-Wire Wire Line
-	1000 1850 1700 1850
-Connection ~ 1100 2350
-Wire Wire Line
-	1100 2550 1100 2150
-Wire Wire Line
-	1700 2350 1700 2550
-Wire Wire Line
-	1700 7300 1700 6000
-Wire Wire Line
-	1700 5800 1700 5600
-Wire Wire Line
-	1700 5400 1100 5400
-Wire Wire Line
-	1100 5400 1100 5800
-Connection ~ 1100 5600
-Wire Wire Line
-	1700 5100 1000 5100
-Wire Wire Line
-	1000 5100 1000 6000
-Wire Wire Line
-	1000 6000 1700 6000
-Connection ~ 1100 6000
-Wire Wire Line
-	1100 2150 1700 2150
-Wire Wire Line
-	1700 2750 1700 4050
-Wire Wire Line
-	1700 4050 2600 4050
-Wire Wire Line
-	2600 7400 2600 7300
-Wire Wire Line
-	5900 1450 5900 1600
-Wire Wire Line
-	4900 1250 5900 1250
-Wire Wire Line
-	4400 1450 3600 1450
-Wire Wire Line
-	1200 1150 1200 1450
-Connection ~ 1200 1150
-Wire Wire Line
-	5100 2350 3600 2350
-Wire Wire Line
-	1700 4700 1700 4300
-Wire Wire Line
-	3600 1850 3750 1850
-Wire Wire Line
-	3750 1850 3750 5100
-Wire Wire Line
-	3600 1650 4000 1650
-Wire Wire Line
-	4000 1650 4000 4300
-Wire Wire Line
-	4000 4300 1700 4300
-Wire Wire Line
-	4400 1650 4300 1650
-Connection ~ 4300 1650
-Wire Wire Line
-	900  4800 900  7300
-Wire Wire Line
-	900  7300 2600 7300
-Connection ~ 1700 7300
-Wire Wire Line
-	900  4400 5900 4400
-Wire Wire Line
-	950  5000 900  5000
-Connection ~ 900  5000
-Wire Wire Line
-	3600 5400 3900 5400
-Wire Wire Line
-	3600 5600 3900 5600
-Wire Wire Line
-	3600 5800 3900 5800
-Wire Wire Line
-	1450 5000 1450 4900
-Wire Wire Line
-	3600 6100 3850 6100
-Wire Wire Line
-	3600 6300 3850 6300
-Wire Wire Line
-	3600 6500 3850 6500
-Wire Wire Line
-	3600 6700 3900 6700
-Wire Wire Line
-	3900 6900 3900 7050
-Wire Wire Line
-	3900 7050 4450 7050
-Wire Wire Line
-	4450 7050 4450 4700
-Wire Wire Line
-	4450 4700 3600 4700
-Wire Wire Line
-	3850 5100 3600 5100
-Connection ~ 3750 5100
-Wire Wire Line
-	3850 4900 3600 4900
+Wire Wire Line
+	3600 1750 3800 1750
+Wire Wire Line
+	3600 1950 3800 1950
+Wire Wire Line
+	3900 4050 3750 4050
+Wire Wire Line
+	3750 4050 3750 5100
+$Comp
+L CONN_3 K?
+U 1 1 56F01643
+P 4250 4050
+F 0 "K?" V 4200 4050 50  0000 C CNN
+F 1 "CONN_3" V 4300 4050 40  0000 C CNN
+	1    4250 4050
+	1    0    0    -1
+$EndComp
+$Comp
+L CONN_3 K?
+U 1 1 56F015E9
+P 4150 1850
+F 0 "K?" V 4100 1850 50  0000 C CNN
+F 1 "CONN_3" V 4200 1850 40  0000 C CNN
+	1    4150 1850
+	1    0    0    -1
+$EndComp
 $Comp
 L CONN_5 P2

Commit message: updated at >>
Parts:
- removed P3: CONN_5, symbol CONN_5
- added P3: CONN_4, symbol CONN_4
- added P5: CONN_2, symbol CONN_2
- added R10, R6, R7, R8, R9: R, symbol R
- gave numbers to parts that had none: 2
Connections:
- wire segments 77 -> 88
Other:
- note added: ">> 5 buttons keyboard"
- note added: ">> display"
- moved on the sheet: P1
