File: layout.sch (KiCad schematic (older format))
At the start: 30 parts, among them IC1 ATMEGA8-P, IC2 ATMEGA8-P, J1 externí zdroj 5V, J2 USB_2, K1 CONN_3, K2 CONN_3, P1 CONN_6, P2 CONN_5, P3 CONN_4, P4 CONN_4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

Commit message: updated at >>
Other:
- note added: ">> 5 butons keybord"
- note removed: ">> 5 buttons keyboard"
Changed lines of the file:
@@
-EESchema Schematic File Version 2  date St 23. březen 2016, 17:05:34 CET
+EESchema Schematic File Version 2  date St 23. březen 2016, 17:13:10 CET
 LIBS:power
 LIBS:device
@@
 Comment4 ""
 $EndDescr
-Text Notes 4850 5700 0    60   ~ 0
->> 5 buttons keyboard
+Text Notes 4450 7300 0    60   ~ 0
+>> display
+Text Notes 4900 5650 0    60   ~ 0
+>> 5 butons keybord
 Wire Wire Line
 	3900 7150 3750 7150
@@
 Wire Wire Line
 	3650 7350 3900 7350
-Text Notes 4450 7300 0    60   ~ 0
->> display
 $Comp
 L CONN_2 P5

Commit message: updated at >>
Parts:
- R10, R6, R7, R8, R9: value R -> 47k
Changed lines of the file:
@@
-EESchema Schematic File Version 2  date St 23. březen 2016, 17:13:10 CET
+EESchema Schematic File Version 2  date St 23. březen 2016, 17:17:15 CET
 LIBS:power
 LIBS:device
@@
 P 3950 5400
 F 0 "R6" V 4030 5400 50  0000 C CNN
-F 1 "R" V 3950 5400 50  0000 C CNN
+F 1 "47k" V 3950 5400 50  0000 C CNN
 	1    3950 5400
 	0    -1   -1   0
@@
 P 3950 5500
 F 0 "R7" V 4030 5500 50  0000 C CNN
-F 1 "R" V 3950 5500 50  0000 C CNN
+F 1 "47k" V 3950 5500 50  0000 C CNN
 	1    3950 5500
 	0    -1   -1   0
@@
 P 3950 5600
 F 0 "R8" V 4030 5600 50  0000 C CNN
-F 1 "R" V 3950 5600 50  0000 C CNN
+F 1 "47k" V 3950 5600 50  0000 C CNN
 	1    3950 5600
 	0    -1   -1   0
@@
 P 3950 5700
 F 0 "R9" V 4030 5700 50  0000 C CNN
-F 1 "R" V 3950 5700 50  0000 C CNN
+F 1 "47k" V 3950 5700 50  0000 C CNN
 	1    3950 5700
 	0    -1   -1   0
@@
 P 3950 6100
 F 0 "R10" V 4030 6100 50  0000 C CNN
-F 1 "R" V 3950 6100 50  0000 C CNN
+F 1 "47k" V 3950 6100 50  0000 C CNN
 	1    3950 6100
 	0    -1   -1   0
