File: layout.sch (KiCad schematic (older format))
At the start: 30 parts, among them IC1 ATMEGA8-P, IC2 ATMEGA8-P, J1 externí zdroj 5V, J2 USB_2, K1 CONN_3, K2 CONN_3, P1 CONN_6, P2 CONN_5, P3 CONN_4, P4 CONN_4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

Commit message: updated at >>
Parts:
- removed JP1: JUMPER-slow_sck, symbol JUMPER
- removed P5: CONN_2, symbol CONN_2
- added P10, P11, P12, P13, P14, P15, P16, P17, P5, P6, P8, P9: CONNECTOR, symbol CONNECTOR
Connections:
- wire segments 88 -> 151
Other:
- moved on the sheet: P1, R10, R3, R6, R7, R8, R9

Commit message: updated at >>
Parts:
- added P? (x2): CONNECTOR, symbol CONNECTOR
Connections:
- wire segments 151 -> 121

Commit message: updated at >>
Other:
- note added: ">> 5 butons keybord I2C port"
- note removed: ">> 5 butons keybord"
Changed lines of the file:
@@
-EESchema Schematic File Version 2  date Út 12. duben 2016, 17:38:28 CEST
+EESchema Schematic File Version 2  date St 25. květen 2016, 12:57:06 CEST
 LIBS:power
 LIBS:device
@@
 Sheet 1 1
 Title ""
-Date "12 apr 2016"
+Date "25 may 2016"
 Rev ""
 Comp ""
@@
 >> display
 Text Notes 5850 6800 0    60   ~ 0
->> 5 butons keybord
+>> 5 butons keybord I2C port
 $Comp
 L R R6

Commit message: updated at >>
Other:
- note added: ">> 5 butons keybord"
- note added: ">> display I2C"
- note removed: ">> 5 butons keybord I2C port"
- note removed: ">> display"
Changed lines of the file:
@@
-EESchema Schematic File Version 2  date St 25. květen 2016, 12:57:06 CEST
+EESchema Schematic File Version 2  date Út 31. květen 2016, 20:32:47 CEST
 LIBS:power
 LIBS:device
@@
 Sheet 1 1
 Title ""
-Date "25 may 2016"
+Date "31 may 2016"
 Rev ""
 Comp ""
@@
 $EndComp
 Text Notes 4450 7300 0    60   ~ 0
->> display
+>> display I2C
 Text Notes 5850 6800 0    60   ~ 0
->> 5 butons keybord I2C port
+>> 5 butons keybord
 $Comp
 L R R6

Commit message: updated at >>
Parts:
- added U1: LM555N, symbol LM555N
- gave numbers to parts that had none: 2
Connections:
- wire segments 121 -> 126

Commit message: updated at >>
Parts:
- removed U1: LM555N, symbol LM555N
- added K3: CONN_3, symbol CONN_3
- added P19, P20, P21, P22, P23, P24, P25, P26, P27, P28: CONNECTOR, symbol CONNECTOR
- added Q1, Q2, Q3, Q4, Q5, Q6, Q7, Q8, Q9: IRF3710, TO220, symbol IRF3710
- added R11, R12, R13, R14, R15, R16, R17, R18, R19: 1k5, symbol R
Connections:
- wire segments 126 -> 176
Other:
- note added: ">> 5 butons keyboard"
- note removed: ">> 5 butons keybord"

Commit message: updated at >>
Parts:
- added P29, P30: CONNECTOR, symbol CONNECTOR
Connections:
- net labels added: Basic usb_asp programmer with apl. circuit - atmega8 + trans.
- net labels removed: Basic usb_asp programmer with apl. circuit - atmega8
- wire segments 176 -> 177
Changed lines of the file:
@@
-EESchema Schematic File Version 2  date Pá 24. únor 2017, 12:04:14 CET
+EESchema Schematic File Version 2  date Pá 24. únor 2017, 18:36:20 CET
 LIBS:power
 LIBS:device
@@
 Comment4 ""
 $EndDescr
+Connection ~ 4900 950
+Wire Wire Line
+	4900 750  4900 1100
 Connection ~ 9250 2550
 Connection ~ 6650 2550
@@
 Wire Wire Line
 	9050 1150 9200 1150
-Wire Wire Line
-	4900 950  4900 1100
 Wire Wire Line
 	4900 1100 5150 1100
@@
 Wire Wire Line
 	6650 2400 6500 2400
+Wire Wire Line
+	5700 1150 5700 750
+Connection ~ 5700 1150
+$Comp
+L CONNECTOR P30
+U 1 1 58B04B82
+P 5700 750
+F 0 "P30" H 6050 850 70  0000 C CNN
+F 1 "CONNECTOR" H 6050 650 70  0000 C CNN
+	1    5700 750
+	1    0    0    -1
+$EndComp
+$Comp
+L CONNECTOR P29
+U 1 1 58B04B79
+P 4900 750
+F 0 "P29" H 5250 850 70  0000 C CNN
+F 1 "CONNECTOR" H 5250 650 70  0000 C CNN
+	1    4900 750
+	1    0    0    -1
+$EndComp
 $Comp
 L CONNECTOR P28
@@
 	1    0    0    -1
 $EndComp
-Text Label 8550 7350 0    60   ~ 0
-Basic usb_asp programmer with apl. circuit - atmega8
+Text Label 8200 7350 0    60   ~ 0
+Basic usb_asp programmer with apl. circuit - atmega8 + trans.
 $Comp
 L GND #PWR03

Commit message: updated at >>
Parts:
- added C6: C, symbol C
- added D2: DIODE, symbol DIODE
- added Q10: 7805, TO220, symbol IRF3710
Connections:
- wire segments 177 -> 189
Other:
- note added: "+12V"
Changed lines of the file:
@@
-EESchema Schematic File Version 2  date Pá 24. únor 2017, 18:36:20 CET
+EESchema Schematic File Version 2  date So 25. únor 2017, 09:10:38 CET
 LIBS:power
 LIBS:device
@@
 EELAYER 25  0
 EELAYER END
-$Descr A4 11700 8267
+$Descr A3 16535 11700
 encoding utf-8
 Sheet 1 1
 Title ""
-Date "24 feb 2017"
+Date "25 feb 2017"
 Rev ""
 Comp ""
@@
 Comment4 ""
 $EndDescr
+Wire Wire Line
+	11400 800  10800 800
+Wire Wire Line
+	10800 1200 10800 1400
+Connection ~ 4800 1150
+Wire Wire Line
+	4800 1150 4800 500
+Wire Wire Line
+	4800 500  11950 500
+Wire Wire Line
+	11950 500  11950 1000
+Connection ~ 6850 1050
+Wire Wire Line
+	6850 650  10400 650
+Wire Wire Line
+	6850 650  6850 1450
 Connection ~ 4900 950
-Wire Wire Line
-	4900 750  4900 1100
 Connection ~ 9250 2550
 Connection ~ 6650 2550
@@
 	9050 1150 9200 1150
 Wire Wire Line
-	4900 1100 5150 1100
+	5150 1100 4900 1100
 Wire Wire Line
 	5150 1100 5150 1450
@@
 Connection ~ 6650 3550
 Wire Wire Line
-	6850 1450 6850 1050
-Wire Wire Line
 	5900 1450 5150 1450
 Wire Wire Line
@@
 	5700 1150 5700 750
 Connection ~ 5700 1150
+Wire Wire Line
+	4900 1100 4900 550
+Wire Wire Line
+	4900 550  10300 550
+Wire Wire Line
+	10300 550  10300 1400
+Wire Wire Line
+	10300 1400 11950 1400
+Connection ~ 10800 1400
+Connection ~ 4900 750
+Wire Wire Line
+	10400 650  10400 1000
+Wire Wire Line
+	10400 1000 10500 1000
+Wire Wire Line
+	11800 800  11950 800
+Connection ~ 11950 800
+$Comp
+L IRF3710 Q10
+U 1 1 58B139B1
+P 10700 1000
+F 0 "Q10" H 10700 852 40  0000 R CNN
+F 1 "7805" H 10700 1149 40  0000 R CNN
+F 2 "TO220" H 10521 1101 29  0000 C CNN
+	1    10700 1000
+	1    0    0    -1
+$EndComp
+Text Notes 6950 800  0    60   ~ 0
++12V
+$Comp
+L C C6
+U 1 1 58B1309A
+P 11950 1200
+F 0 "C6" H 12000 1300 50  0000 L CNN
+F 1 "C" H 12000 1100 50  0000 L CNN
+	1    11950 1200
+	1    0    0    -1
+$EndComp
+$Comp
+L DIODE D2
+U 1 1 58B12F6B
+P 11600 800
+F 0 "D2" H 11600 900 40  0000 C CNN
+F 1 "DIODE" H 11600 700 40  0000 C CNN
+	1    11600 800
+	1    0    0    -1
+$EndComp
 $Comp
 L CONNECTOR P30
@@
 	1    0    0    -1
 $EndComp
-Text Label 8200 7350 0    60   ~ 0
+Text Label 12800 10800 0    60   ~ 0
 Basic usb_asp programmer with apl. circuit - atmega8 + trans.
 $Comp
