File: $layout.sch (KiCad schematic (older format))
At the start: 30 parts, among them IC1 ATMEGA8-P, IC2 ATMEGA8-P, J1 externí zdroj 5V, J2 USB_2, K1 CONN_3, K2 CONN_3, P1 CONN_6, P2 CONN_5, P3 CONN_4, P4 CONN_4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

Commit message: updated at >>
Parts:
- added P6, P7, P8, P9, P? (x2): CONNECTOR, symbol CONNECTOR
Connections:
- wire segments 88 -> 102
Other:
- moved on the sheet: R3
Changed lines of the file:
@@
-EESchema Schematic File Version 2  date St 23. březen 2016, 19:55:29 CET
+EESchema Schematic File Version 2  date Čt 24. březen 2016, 21:10:52 CET
 LIBS:power
 LIBS:device
@@
 Sheet 1 1
 Title ""
-Date "23 mar 2016"
+Date "24 mar 2016"
 Rev ""
 Comp ""
@@
 Comment4 ""
 $EndDescr
-Connection ~ 4750 5700
-Wire Wire Line
-	4750 5700 4750 6700
+Connection ~ 4900 1250
+Wire Wire Line
+	4450 1250 5900 1250
+Connection ~ 2750 1150
+Wire Wire Line
+	2750 1150 2750 1250
+Wire Wire Line
+	2750 1250 2800 1250
+Wire Wire Line
+	4500 2750 4300 2750
+Wire Wire Line
+	4300 2750 4300 1550
+Wire Wire Line
+	5250 7000 5050 7000
+Wire Wire Line
+	5050 7000 5050 7100
+Wire Wire Line
+	5050 7100 5750 7100
+Wire Wire Line
+	5750 7100 5750 5500
+Wire Wire Line
+	5750 5500 5900 5500
+Wire Wire Line
+	4900 6100 3600 6100
+Connection ~ 4650 6100
+Wire Wire Line
+	4650 6100 4650 6900
+Wire Wire Line
+	4650 6900 5250 6900
+Connection ~ 4750 5600
+Wire Wire Line
+	4750 5600 4750 6700
 Wire Wire Line
 	4750 6700 5250 6700
@@
 	5900 4700 5900 4900
 Wire Wire Line
-	3600 3050 4300 3050
-Wire Wire Line
 	4900 1650 5000 1650
 Wire Wire Line
 	5000 1650 5000 1350
 Wire Wire Line
-	4300 3050 4300 1550
-Wire Wire Line
-	4300 1550 3600 1550
-Wire Wire Line
 	5700 2350 5700 2500
 Wire Wire Line
 	5000 1350 5900 1350
 Wire Wire Line
-	4900 1450 4900 1250
-Connection ~ 4400 1150
-Wire Wire Line
-	4400 1150 4400 1250
+	4900 1250 4900 1450
 Connection ~ 2600 1150
 Wire Wire Line
@@
 	5900 1450 5900 1600
 Wire Wire Line
-	4900 1250 5900 1250
-Wire Wire Line
 	4400 1450 3600 1450
 Wire Wire Line
@@
 	4000 4300 1700 4300
 Wire Wire Line
-	4400 1650 4300 1650
+	4300 1650 4400 1650
 Connection ~ 4300 1650
 Wire Wire Line
@@
 Connection ~ 5400 5700
 Wire Wire Line
-	4900 6100 3600 6100
-Wire Wire Line
 	4900 5600 3600 5600
 Wire Wire Line
@@
 	4800 6600 4800 5500
 Connection ~ 4800 5500
-$Comp
-L GND #PWR?
+Wire Wire Line
+	5250 6800 4700 6800
+Wire Wire Line
+	4700 6800 4700 5700
+Connection ~ 4700 5700
+Connection ~ 5750 4400
+Wire Wire Line
+	5900 5200 5750 5200
+Wire Wire Line
+	5750 5200 5750 4400
+Wire Wire Line
+	4300 1550 3600 1550
+Wire Wire Line
+	4500 3050 3600 3050
+Wire Wire Line
+	3300 1250 3500 1250
+$Comp
+L CONNECTOR P?
+U 1 1 56F44736
+P 4450 1250
+F 0 "P?" H 4800 1350 70  0000 C CNN
+F 1 "CONNECTOR" H 4800 1150 70  0000 C CNN
+	1    4450 1250
+	-1   0    0    -1
+$EndComp
+$Comp
+L CONNECTOR P?
+U 1 1 56F4472A
+P 3500 1250
+F 0 "P?" H 3850 1350 70  0000 C CNN
+F 1 "CONNECTOR" H 3850 1150 70  0000 C CNN
+	1    3500 1250
+	1    0    0    -1
+$EndComp
+$Comp
+L CONNECTOR P9
+U 1 1 56F4451F
+P 4500 3050
+F 0 "P9" H 4850 3150 70  0000 C CNN
+F 1 "CONNECTOR" H 4850 2950 70  0000 C CNN
+	1    4500 3050
+	1    0    0    -1
+$EndComp
+$Comp
+L CONNECTOR P8
+U 1 1 56F44512
+P 4500 2750
+F 0 "P8" H 4850 2850 70  0000 C CNN
+F 1 "CONNECTOR" H 4850 2650 70  0000 C CNN
+	1    4500 2750
+	1    0    0    -1
+$EndComp
+$Comp
+L CONNECTOR P7
+U 1 1 56F43F14
+P 5900 5500
+F 0 "P7" H 6250 5600 70  0000 C CNN
+F 1 "CONNECTOR" H 6250 5400 70  0000 C CNN
+	1    5900 5500
+	1    0    0    -1
+$EndComp
+$Comp
+L CONNECTOR P6
+U 1 1 56F43F05
+P 5900 5200
+F 0 "P6" H 6250 5300 70  0000 C CNN
+F 1 "CONNECTOR" H 6250 5100 70  0000 C CNN
+	1    5900 5200
+	1    0    0    -1
+$EndComp
+$Comp
+L GND #PWR3
 U 1 1 56F2E64F
 P 5400 6250
-F 0 "#PWR?" H 5400 6250 30  0001 C CNN
+F 0 "#PWR3" H 5400 6250 30  0001 C CNN
 F 1 "GND" H 5400 6180 30  0001 C CNN
 	1    5400 6250
@@
 Text Notes 4450 7300 0    60   ~ 0
 >> display
-Text Notes 6250 6250 0    60   ~ 0
+Text Notes 5850 6800 0    60   ~ 0
 >> 5 butons keybord
 $Comp
@@
 Basic usb_asp programmer with apl. circuit - atmega8
 $Comp
-L GND #PWR01
+L GND #PWR6
 U 1 1 56E6FC1F
 P 5900 4900
-F 0 "#PWR01" H 5900 4900 30  0001 C CNN
+F 0 "#PWR6" H 5900 4900 30  0001 C CNN
 F 1 "GND" H 5900 4830 30  0001 C CNN
 	1    5900 4900
@@
 $EndComp
 $Comp
-L GND #PWR02
+L GND #PWR4
 U 1 1 56E6F74F
 P 5700 2500
-F 0 "#PWR02" H 5700 2500 30  0001 C CNN
+F 0 "#PWR4" H 5700 2500 30  0001 C CNN
 F 1 "GND" H 5700 2430 30  0001 C CNN
 	1    5700 2500
@@
 $EndComp
 $Comp
-L GND #PWR03
+L GND #PWR5
 U 1 1 56E6F4BB
 P 5900 1600
-F 0 "#PWR03" H 5900 1600 30  0001 C CNN
+F 0 "#PWR5" H 5900 1600 30  0001 C CNN
 F 1 "GND" H 5900 1530 30  0001 C CNN
 	1    5900 1600
@@
 L R R3
 U 1 1 56E6F06F
-P 4650 1250
-F 0 "R3" V 4730 1250 50  0000 C CNN
-F 1 "10k" V 4650 1250 50  0000 C CNN
-	1    4650 1250
+P 3050 1250
+F 0 "R3" V 3130 1250 50  0000 C CNN
+F 1 "10k" V 3050 1250 50  0000 C CNN
+	1    3050 1250
 	0    -1   -1   0
 $EndComp
@@
 $EndComp
 $Comp
-L GND #PWR04
+L GND #PWR1
 U 1 1 56E6EE76
 P 2600 4150
-F 0 "#PWR04" H 2600 4150 30  0001 C CNN
+F 0 "#PWR1" H 2600 4150 30  0001 C CNN
 F 1 "GND" H 2600 4080 30  0001 C CNN
 	1    2600 4150
@@
 $EndComp
 $Comp
-L GND #PWR05
+L GND #PWR2
 U 1 1 56E6ED32
 P 2600 7400
-F 0 "#PWR05" H 2600 7400 30  0001 C CNN
+F 0 "#PWR2" H 2600 7400 30  0001 C CNN
 F 1 "GND" H 2600 7330 30  0001 C CNN
 	1    2600 7400

Commit message: updated at >>
Parts:
- removed JP1: JUMPER-slow_sck, symbol JUMPER
- added P12, P13, P14, P15, P16, P17: CONNECTOR, symbol CONNECTOR
- gave numbers to parts that had none: 2
Connections:
- wire segments 102 -> 110
Changed lines of the file:
@@
-EESchema Schematic File Version 2  date Čt 24. březen 2016, 21:10:52 CET
+EESchema Schematic File Version 2  date Čt 24. březen 2016, 23:12:19 CET
 LIBS:power
 LIBS:device
@@
 Comment4 ""
 $EndDescr
+Wire Wire Line
+	900  3950 900  4450
+Wire Wire Line
+	900  3050 900  1150
+Wire Wire Line
+	4500 2350 4500 2450
+Wire Wire Line
+	6050 1850 5700 1850
+Wire Wire Line
+	5900 1250 5700 1250
+Wire Wire Line
+	5700 1250 5700 1850
 Connection ~ 4900 1250
-Wire Wire Line
-	4450 1250 5900 1250
 Connection ~ 2750 1150
 Wire Wire Line
@@
 	5750 5500 5900 5500
 Wire Wire Line
-	4900 6100 3600 6100
+	3600 6100 4900 6100
 Connection ~ 4650 6100
 Wire Wire Line
@@
 	4850 6500 5250 6500
 Wire Wire Line
-	4900 5500 3600 5500
-Wire Wire Line
-	4900 5700 3600 5700
+	3600 5500 4900 5500
+Wire Wire Line
+	3600 5700 4900 5700
 Connection ~ 5400 6100
 Wire Wire Line
-	5400 6250 5400 5400
+	5400 5400 5400 6250
 Connection ~ 5400 5500
 Connection ~ 5400 5600
@@
 Wire Wire Line
 	3600 1750 3800 1750
-Wire Wire Line
-	3850 4800 3600 4800
 Connection ~ 3700 5000
 Wire Wire Line
-	3600 5000 3850 5000
+	3850 5000 3600 5000
 Connection ~ 3800 5200
 Wire Wire Line
-	3600 5200 3850 5200
+	3850 5200 3600 5200
 Wire Wire Line
 	3600 6800 3900 6800
@@
 Connection ~ 1450 4400
 Wire Wire Line
-	1450 4400 1450 4500
+	1450 4500 1450 4400
 Connection ~ 900  4400
 Connection ~ 2600 4400
 Wire Wire Line
-	900  4450 900  1150
-Wire Wire Line
 	5900 4700 5900 4900
 Wire Wire Line
@@
 Wire Wire Line
 	5000 1650 5000 1350
-Wire Wire Line
-	5700 2350 5700 2500
 Wire Wire Line
 	5000 1350 5900 1350
@@
 Connection ~ 1200 1150
 Wire Wire Line
-	5100 2350 3600 2350
-Wire Wire Line
 	1700 4700 1700 4300
 Wire Wire Line
@@
 	4000 4300 1700 4300
 Wire Wire Line
-	4300 1650 4400 1650
+	4400 1650 4300 1650
 Connection ~ 4300 1650
 Wire Wire Line
@@
 Connection ~ 1700 7300
 Wire Wire Line
-	5900 4400 900  4400
-Wire Wire Line
-	900  5000 950  5000
+	950  5000 900  5000
 Connection ~ 900  5000
 Wire Wire Line
@@
 	4450 4700 3600 4700
 Wire Wire Line
-	3600 5100 3850 5100
+	3850 5100 3600 5100
 Connection ~ 3750 5100
 Wire Wire Line
@@
 Connection ~ 5400 5700
 Wire Wire Line
-	4900 5600 3600 5600
-Wire Wire Line
-	4900 5400 3600 5400
+	3600 5600 4900 5600
+Wire Wire Line
+	3600 5400 4900 5400
 Wire Wire Line
 	5250 6600 4800 6600
@@
 Wire Wire Line
 	3300 1250 3500 1250
-$Comp
-L CONNECTOR P?
+Wire Wire Line
+	3850 4800 3600 4800
+Wire Wire Line
+	6050 2150 5600 2150
+Wire Wire Line
+	5600 2150 5600 1250
+Wire Wire Line
+	5600 1250 4450 1250
+Wire Wire Line
+	3600 2350 4400 2350
+Wire Wire Line
+	4400 2350 4400 2050
+Wire Wire Line
+	4400 2050 4500 2050
+Wire Wire Line
+	900  4400 5900 4400
+$Comp
+L CONNECTOR P16
+U 1 1 56F463EF
+P 900 3050
+F 0 "P16" H 1250 3150 70  0000 C CNN
+F 1 "CONNECTOR" H 1250 2950 70  0000 C CNN
+	1    900  3050
+	0    1    1    0
+$EndComp
+$Comp
+L CONNECTOR P17
+U 1 1 56F463EA
+P 900 3950
+F 0 "P17" H 1250 4050 70  0000 C CNN
+F 1 "CONNECTOR" H 1250 3850 70  0000 C CNN
+	1    900  3950
+	0    -1   -1   0
+$EndComp
+$Comp
+L CONNECTOR P14
+U 1 1 56F4532C
+P 4500 2050
+F 0 "P14" H 4850 2150 70  0000 C CNN
+F 1 "CONNECTOR" H 4850 1950 70  0000 C CNN
+	1    4500 2050
+	1    0    0    -1
+$EndComp
+$Comp
+L CONNECTOR P15
+U 1 1 56F45321
+P 4500 2350
+F 0 "P15" H 4850 2450 70  0000 C CNN
+F 1 "CONNECTOR" H 4850 2250 70  0000 C CNN
+	1    4500 2350
+	1    0    0    -1
+$EndComp
+$Comp
+L CONNECTOR P12
+U 1 1 56F4507E
+P 6050 1850
+F 0 "P12" H 6400 1950 70  0000 C CNN
+F 1 "CONNECTOR" H 6400 1750 70  0000 C CNN
+	1    6050 1850
+	1    0    0    -1
+$EndComp
+$Comp
+L CONNECTOR P13
+U 1 1 56F45079
+P 6050 2150
+F 0 "P13" H 6400 2250 70  0000 C CNN
+F 1 "CONNECTOR" H 6400 2050 70  0000 C CNN
+	1    6050 2150
+	1    0    0    -1
+$EndComp
+$Comp
+L CONNECTOR P11
 U 1 1 56F44736
 P 4450 1250
-F 0 "P?" H 4800 1350 70  0000 C CNN
+F 0 "P11" H 4800 1350 70  0000 C CNN
 F 1 "CONNECTOR" H 4800 1150 70  0000 C CNN
 	1    4450 1250
@@
 $EndComp
 $Comp
-L CONNECTOR P?
+L CONNECTOR P10
 U 1 1 56F4472A
 P 3500 1250
-F 0 "P?" H 3850 1350 70  0000 C CNN
+F 0 "P10" H 3850 1350 70  0000 C CNN
 F 1 "CONNECTOR" H 3850 1150 70  0000 C CNN
 	1    3500 1250
@@
 $EndComp
 $Comp
-L GND #PWR3
+L GND #PWR4
 U 1 1 56F2E64F
 P 5400 6250
-F 0 "#PWR3" H 5400 6250 30  0001 C CNN
+F 0 "#PWR4" H 5400 6250 30  0001 C CNN
 F 1 "GND" H 5400 6180 30  0001 C CNN
 	1    5400 6250
@@
 $EndComp
 $Comp
-L GND #PWR4
+L GND #PWR3
 U 1 1 56E6F74F
-P 5700 2500
-F 0 "#PWR4" H 5700 2500 30  0001 C CNN
-F 1 "GND" H 5700 2430 30  0001 C CNN
-	1    5700 2500
-	1    0    0    -1
-$EndComp
-$Comp
-L JUMPER JP1
-U 1 1 56E6F717
-P 5400 2350
-F 0 "JP1" H 5400 2500 60  0000 C CNN
-F 1 "JUMPER-slow_sck" H 5400 2270 40  0000 C CNN
-	1    5400 2350
-	1    0    0    -1
-$EndComp
+P 4500 2450
+F 0 "#PWR3" H 4500 2450 30  0001 C CNN
+F 1 "GND" H 4500 2380 30  0001 C CNN
+	1    4500 2450
+	1    0    0    -1
+$EndComp

Commit message: updated at >>
Parts:
- removed P6, P7: CONNECTOR, symbol CONNECTOR
Connections:
- wire segments 110 -> 115
Other:
- moved on the sheet: P1
Changed lines of the file:
@@
-EESchema Schematic File Version 2  date Čt 24. březen 2016, 23:12:19 CET
+EESchema Schematic File Version 2  date Pá 25. březen 2016, 07:58:06 CET
 LIBS:power
 LIBS:device
@@
 Sheet 1 1
 Title ""
-Date "24 mar 2016"
+Date "25 mar 2016"
 Rev ""
 Comp ""
@@
 $EndDescr
 Wire Wire Line
+	5250 7100 4650 7100
+Wire Wire Line
+	4650 7100 4650 6100
+Wire Wire Line
+	5250 6900 4750 6900
+Wire Wire Line
+	4750 6900 4750 5600
+Wire Wire Line
+	5250 6700 4850 6700
+Wire Wire Line
+	4850 6700 4850 5400
+Connection ~ 900  2850
+Wire Wire Line
+	900  2850 600  2850
+Wire Wire Line
+	600  2850 600  4150
+Connection ~ 900  4150
+Wire Wire Line
+	600  4150 900  4150
+Connection ~ 4400 3050
+Connection ~ 4400 2750
+Wire Wire Line
+	4400 3050 4400 2750
+Connection ~ 3400 1250
+Wire Wire Line
+	3400 1250 3400 950
+Wire Wire Line
+	3400 950  4600 950
+Connection ~ 4600 1250
+Wire Wire Line
+	4600 950  4600 1250
+Wire Wire Line
 	900  3950 900  4450
 Wire Wire Line
 	900  3050 900  1150
-Wire Wire Line
-	4500 2350 4500 2450
 Wire Wire Line
 	6050 1850 5700 1850
@@
 	4300 2750 4300 1550
 Wire Wire Line
-	5250 7000 5050 7000
-Wire Wire Line
-	5050 7000 5050 7100
-Wire Wire Line
-	5050 7100 5750 7100
-Wire Wire Line
-	5750 7100 5750 5500
-Wire Wire Line
-	5750 5500 5900 5500
-Wire Wire Line
 	3600 6100 4900 6100
 Connection ~ 4650 6100
-Wire Wire Line
-	4650 6100 4650 6900
-Wire Wire Line
-	4650 6900 5250 6900
 Connection ~ 4750 5600
-Wire Wire Line
-	4750 5600 4750 6700
-Wire Wire Line
-	4750 6700 5250 6700
 Connection ~ 4850 5400
-Wire Wire Line
-	4850 5400 4850 6500
-Wire Wire Line
-	4850 6500 5250 6500
 Wire Wire Line
 	3600 5500 4900 5500
@@
 Wire Wire Line
 	3600 5400 4900 5400
-Wire Wire Line
-	5250 6600 4800 6600
-Wire Wire Line
-	4800 6600 4800 5500
 Connection ~ 4800 5500
-Wire Wire Line
-	5250 6800 4700 6800
-Wire Wire Line
-	4700 6800 4700 5700
 Connection ~ 4700 5700
 Connection ~ 5750 4400
 Wire Wire Line
-	5900 5200 5750 5200
-Wire Wire Line
-	5750 5200 5750 4400
-Wire Wire Line
 	4300 1550 3600 1550
 Wire Wire Line
@@
 Wire Wire Line
 	900  4400 5900 4400
+Wire Wire Line
+	5700 1650 5600 1650
+Connection ~ 5600 1650
+Connection ~ 5700 1650
+Wire Wire Line
+	4500 2050 4500 2450
+Connection ~ 4500 2350
+Wire Wire Line
+	5750 4400 5750 6450
+Wire Wire Line
+	5750 6450 5150 6450
+Wire Wire Line
+	5150 6450 5150 6600
+Wire Wire Line
+	5150 6600 5250 6600
+Wire Wire Line
+	4800 5500 4800 6800
+Wire Wire Line
+	4800 6800 5250 6800
+Wire Wire Line
+	4700 5700 4700 7000
+Wire Wire Line
+	4700 7000 5250 7000
 $Comp
 L CONNECTOR P16
@@
 $EndComp
 $Comp
-L CONNECTOR P7
-U 1 1 56F43F14
-P 5900 5500
-F 0 "P7" H 6250 5600 70  0000 C CNN
-F 1 "CONNECTOR" H 6250 5400 70  0000 C CNN
-	1    5900 5500
-	1    0    0    -1
-$EndComp
-$Comp
-L CONNECTOR P6
-U 1 1 56F43F05
-P 5900 5200
-F 0 "P6" H 6250 5300 70  0000 C CNN
-F 1 "CONNECTOR" H 6250 5100 70  0000 C CNN
-	1    5900 5200
-	1    0    0    -1
-$EndComp
-$Comp
-L GND #PWR4
+L GND #PWR01
 U 1 1 56F2E64F
 P 5400 6250
-F 0 "#PWR4" H 5400 6250 30  0001 C CNN
+F 0 "#PWR01" H 5400 6250 30  0001 C CNN
 F 1 "GND" H 5400 6180 30  0001 C CNN
 	1    5400 6250
@@
 L CONN_6 P1
 U 1 1 56EABEA5
-P 5600 6750
-F 0 "P1" V 5550 6750 60  0000 C CNN
-F 1 "CONN_6" V 5650 6750 60  0000 C CNN
-	1    5600 6750
+P 5600 6850
+F 0 "P1" V 5550 6850 60  0000 C CNN
+F 1 "CONN_6" V 5650 6850 60  0000 C CNN
+	1    5600 6850
 	1    0    0    -1
 $EndComp
@@
 Basic usb_asp programmer with apl. circuit - atmega8
 $Comp
-L GND #PWR6
+L GND #PWR02
 U 1 1 56E6FC1F
 P 5900 4900
-F 0 "#PWR6" H 5900 4900 30  0001 C CNN
+F 0 "#PWR02" H 5900 4900 30  0001 C CNN
 F 1 "GND" H 5900 4830 30  0001 C CNN
 	1    5900 4900
@@
 $EndComp
 $Comp
-L GND #PWR3
+L GND #PWR03
 U 1 1 56E6F74F
 P 4500 2450
-F 0 "#PWR3" H 4500 2450 30  0001 C CNN
+F 0 "#PWR03" H 4500 2450 30  0001 C CNN
 F 1 "GND" H 4500 2380 30  0001 C CNN
 	1    4500 2450
@@
 $EndComp
 $Comp
-L GND #PWR5
+L GND #PWR04
 U 1 1 56E6F4BB
 P 5900 1600
-F 0 "#PWR5" H 5900 1600 30  0001 C CNN
+F 0 "#PWR04" H 5900 1600 30  0001 C CNN
 F 1 "GND" H 5900 1530 30  0001 C CNN
 	1    5900 1600
@@
 $EndComp
 $Comp
-L GND #PWR1
+L GND #PWR05
 U 1 1 56E6EE76
 P 2600 4150
-F 0 "#PWR1" H 2600 4150 30  0001 C CNN
+F 0 "#PWR05" H 2600 4150 30  0001 C CNN
 F 1 "GND" H 2600 4080 30  0001 C CNN
 	1    2600 4150
@@
 $EndComp
 $Comp
-L GND #PWR2
+L GND #PWR06
 U 1 1 56E6ED32
 P 2600 7400
-F 0 "#PWR2" H 2600 7400 30  0001 C CNN
+F 0 "#PWR06" H 2600 7400 30  0001 C CNN
 F 1 "GND" H 2600 7330 30  0001 C CNN
 	1    2600 7400

Commit message: updated at >>
Parts:
- removed P5: CONN_2, symbol CONN_2
- added P5, P6: CONNECTOR, symbol CONNECTOR
Changed lines of the file:
@@
-EESchema Schematic File Version 2  date Pá 25. březen 2016, 07:58:06 CET
+EESchema Schematic File Version 2  date Pá 25. březen 2016, 09:02:57 CET
 LIBS:power
 LIBS:device
@@
 Comment4 ""
 $EndDescr
+$Comp
+L CONNECTOR P6
+U 1 1 56F4EE63
+P 3900 7350
+F 0 "P6" H 4250 7450 70  0000 C CNN
+F 1 "CONNECTOR" H 4250 7250 70  0000 C CNN
+	1    3900 7350
+	1    0    0    -1
+$EndComp
+$Comp
+L CONNECTOR P5
+U 1 1 56F4EE5E
+P 3900 7150
+F 0 "P5" H 4250 7250 70  0000 C CNN
+F 1 "CONNECTOR" H 4250 7050 70  0000 C CNN
+	1    3900 7150
+	1    0    0    -1
+$EndComp
 Wire Wire Line
 	5250 7100 4650 7100
@@
 >> 5 butons keybord
 $Comp
-L CONN_2 P5
-U 1 1 56F2B9DF
-P 4250 7250
-F 0 "P5" V 4200 7250 40  0000 C CNN
-F 1 "CONN_2" V 4300 7250 40  0000 C CNN
-	1    4250 7250
-	1    0    0    -1
-$EndComp
-$Comp
 L R R6

Commit message: updated at >>
Connections:
- wire segments 115 -> 151
Changed lines of the file:
@@
-EESchema Schematic File Version 2  date Pá 25. březen 2016, 09:02:57 CET
+EESchema Schematic File Version 2  date Pá 25. březen 2016, 09:15:00 CET
 LIBS:power
 LIBS:device
@@
 Connection ~ 900  2850
 Wire Wire Line
-	900  2850 600  2850
-Wire Wire Line
-	600  2850 600  4150
+	900  2850 700  2850
+Wire Wire Line
+	700  2850 700  4150
 Connection ~ 900  4150
 Wire Wire Line
-	600  4150 900  4150
+	700  4150 900  4150
 Connection ~ 4400 3050
 Connection ~ 4400 2750
@@
 	4600 950  4600 1250
 Wire Wire Line
-	900  3950 900  4450
-Wire Wire Line
-	900  3050 900  1150
+	900  3950 900  4150
+Wire Wire Line
+	900  4150 900  4400
+Wire Wire Line
+	900  4400 900  4450
+Wire Wire Line
+	900  3050 900  2850
+Wire Wire Line
+	900  2850 900  1150
 Wire Wire Line
 	6050 1850 5700 1850
@@
 	5900 1250 5700 1250
 Wire Wire Line
-	5700 1250 5700 1850
+	5700 1250 5700 1650
+Wire Wire Line
+	5700 1650 5700 1850
 Connection ~ 4900 1250
 Connection ~ 2750 1150
@@
 	2750 1250 2800 1250
 Wire Wire Line
-	4500 2750 4300 2750
-Wire Wire Line
-	4300 2750 4300 1550
-Wire Wire Line
-	3600 6100 4900 6100
+	4500 2750 4400 2750
+Wire Wire Line
+	4400 2750 4300 2750
+Wire Wire Line
+	4300 2750 4300 1650
+Wire Wire Line
+	4300 1650 4300 1550
+Wire Wire Line
+	3600 6100 4650 6100
+Wire Wire Line
+	4650 6100 4900 6100
 Connection ~ 4650 6100
 Connection ~ 4750 5600
 Connection ~ 4850 5400
 Wire Wire Line
-	3600 5500 4900 5500
-Wire Wire Line
-	3600 5700 4900 5700
+	3600 5500 4800 5500
+Wire Wire Line
+	4800 5500 4900 5500
+Wire Wire Line
+	3600 5700 4700 5700
+Wire Wire Line
+	4700 5700 4900 5700
 Connection ~ 5400 6100
 Wire Wire Line
-	5400 5400 5400 6250
+	5400 5400 5400 5500
+Wire Wire Line
+	5400 5500 5400 5600
+Wire Wire Line
+	5400 5600 5400 5700
+Wire Wire Line
+	5400 5700 5400 6100
+Wire Wire Line
+	5400 6100 5400 6250
 Connection ~ 5400 5500
 Connection ~ 5400 5600
 Wire Wire Line
-	900  4850 900  7300
+	900  4850 900  5000
+Wire Wire Line
+	900  5000 900  7300
 Wire Wire Line
 	3900 7150 3750 7150
@@
 Connection ~ 3700 5000
 Wire Wire Line
-	3850 5000 3600 5000
+	3850 5000 3700 5000
+Wire Wire Line
+	3700 5000 3600 5000
 Connection ~ 3800 5200
 Wire Wire Line
-	3850 5200 3600 5200
+	3850 5200 3800 5200
+Wire Wire Line
+	3800 5200 3600 5200
 Wire Wire Line
 	3600 6800 3900 6800
@@
 Connection ~ 2600 1150
 Wire Wire Line
-	900  1150 5900 1150
+	900  1150 1200 1150
+Wire Wire Line
+	1200 1150 2600 1150
+Wire Wire Line
+	2600 1150 2750 1150
+Wire Wire Line
+	2750 1150 5900 1150
 Wire Wire Line
 	2600 4150 2600 4050
 Connection ~ 1100 2750
 Wire Wire Line
-	1000 2750 1700 2750
+	1000 2750 1100 2750
+Wire Wire Line
+	1100 2750 1700 2750
 Wire Wire Line
 	1000 2750 1000 1850
@@
 Connection ~ 1100 2350
 Wire Wire Line
-	1100 2550 1100 2150
+	1100 2550 1100 2350
+Wire Wire Line
+	1100 2350 1100 2150
 Wire Wire Line
 	1700 2350 1700 2550
@@
 	1700 5400 1100 5400
 Wire Wire Line
-	1100 5400 1100 5800
+	1100 5400 1100 5600
+Wire Wire Line
+	1100 5600 1100 5800
 Connection ~ 1100 5600
 Wire Wire Line
@@
 	1000 5100 1000 6000
 Wire Wire Line
-	1000 6000 1700 6000
+	1000 6000 1100 6000
+Wire Wire Line
+	1100 6000 1700 6000
 Connection ~ 1100 6000
 Wire Wire Line
@@
 Connection ~ 4300 1650
 Wire Wire Line
-	2600 7300 900  7300
+	2600 7300 1700 7300
+Wire Wire Line
+	1700 7300 900  7300
 Connection ~ 1700 7300
 Wire Wire Line
@@
 	4450 4700 3600 4700
 Wire Wire Line
-	3850 5100 3600 5100
+	3850 5100 3750 5100
+Wire Wire Line
+	3750 5100 3600 5100
 Connection ~ 3750 5100
 Wire Wire Line
@@
 Connection ~ 5400 5700
 Wire Wire Line
-	3600 5600 4900 5600
-Wire Wire Line
-	3600 5400 4900 5400
+	3600 5600 4750 5600
+Wire Wire Line
+	4750 5600 4900 5600
+Wire Wire Line
+	3600 5400 4850 5400
+Wire Wire Line
+	4850 5400 4900 5400
 Connection ~ 4800 5500
 Connection ~ 4700 5700
@@
 	4300 1550 3600 1550
 Wire Wire Line
-	4500 3050 3600 3050
-Wire Wire Line
-	3300 1250 3500 1250
+	4500 3050 4400 3050
+Wire Wire Line
+	4400 3050 3600 3050
+Wire Wire Line
+	3300 1250 3400 1250
+Wire Wire Line
+	3400 1250 3500 1250
 Wire Wire Line
 	3850 4800 3600 4800
@@
 	6050 2150 5600 2150
 Wire Wire Line
-	5600 2150 5600 1250
-Wire Wire Line
-	5600 1250 4450 1250
+	5600 2150 5600 1650
+Wire Wire Line
+	5600 1650 5600 1250
+Wire Wire Line
+	5600 1250 4900 1250
+Wire Wire Line
+	4900 1250 4600 1250
+Wire Wire Line
+	4600 1250 4450 1250
 Wire Wire Line
 	3600 2350 4400 2350
@@
 	4400 2050 4500 2050
 Wire Wire Line
-	900  4400 5900 4400
+	900  4400 1450 4400
+Wire Wire Line
+	1450 4400 2600 4400
+Wire Wire Line
+	2600 4400 5750 4400
+Wire Wire Line
+	5750 4400 5900 4400
 Wire Wire Line
 	5700 1650 5600 1650
@@
 Connection ~ 5700 1650
 Wire Wire Line
-	4500 2050 4500 2450
+	4500 2050 4500 2350
+Wire Wire Line
+	4500 2350 4500 2450
 Connection ~ 4500 2350
 Wire Wire Line
