File: $layout.sch (KiCad schematic (older format))
At the start: 43 parts, among them IC1 ATMEGA8-P, IC2 ATMEGA8-P, J1 externí zdroj 5V, J2 USB_2, K1 CONN_3, K2 CONN_3, P1 CONN_6, P10 CONNECTOR, P11 CONNECTOR, P12 CONNECTOR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

Commit message: updated at >>
Parts:
- removed U1: LM555N, symbol LM555N
- added K3: CONN_3, symbol CONN_3
- added P19, P20, P21, P22, P23, P24, P25, P26, P27, P28, P29, P30: CONNECTOR, symbol CONNECTOR
- added Q1, Q2, Q3, Q4, Q5, Q6, Q7, Q8, Q9: IRF3710, TO220, symbol IRF3710
- added R11, R12, R13, R14, R15, R16, R17, R18, R19: 1k5, symbol R
Connections:
- wire segments 121 -> 177
Other:
- note added: ">> 5 butons keyboard"
- note removed: ">> 5 butons keybord"
